File: panel_rp2354_20x20_v0p2/drivers.kicad_sch (KiCad schematic)
At the start: 96 parts, among them U10 UCC27517, U11 UCC27517, U12 UCC27517, U13 UCC27517, U14 UCC27517, U15 UCC27517, U16 UCC27517, U17 UCC27517, U18 UCC27517, U19 UCC27517, U20 UCC27517, U21 UCC27517, U22 UCC27517, U23 UCC27517, U24 UCC27517, U25 UCC27517, U26 UCC27517, U27 UCC27517, U28 UCC27517, U29 UCC27517, U3 UCC27517, U30 UCC27517, U31 UCC27517, U32 UCC27517, U33 UCC27517, U34 UCC27517, U35 UCC27517, U36 UCC27517, U37 UCC27517, U38 UCC27517, U39 UCC27517, U4 UCC27517, U40 UCC27517, U41 UCC27517, U42 UCC27517, U5 UCC27517, U6 UCC27517, U7 UCC27517, U8 UCC27517, U9 UCC27517

Commit message: Fixed ERC and DRC warnings
Parts:
- C19, C20, C21, C22, C23, C24, C25, C26, C27, C28, C29, C30, C31, C32, C33, C34, C35, C36, C37, C38, C39, C40, C41, C42, C43, C44, C45, C46, C47, C48, C49, C50, C51, C52, C53, C54, C55, C56, C57, C58: footprint Capacitor_SMD:C_0201_0603Metric -> panel_custom:C_0201_0603Metric
- C59: footprint Capacitor_SMD:C_0402_1005Metric -> panel_custom:C_0402_1005Metric_C61
- C60, C61, C62, C64, C65, C66, C69, C70, C71, C72, C73, C74, C75, C76: footprint Capacitor_SMD:C_0402_1005Metric -> panel_custom:C_0402_1005Metric
- C63: footprint Capacitor_SMD:C_0402_1005Metric -> panel_custom:C_0402_1005Metric_C70
- U10, U11, U12, U13, U14, U15, U16, U17, U18, U19, U20, U21, U22, U23, U24, U25, U26, U27, U28, U29, U3, U30, U31, U32, U33, U34, U35, U36, U37, U38, U39, U4, U40, U41, U42, U5, U6, U7, U8, U9: footprint Package_TO_SOT_SMD:SOT-23-5 -> panel_custom:UCC27517_SOT-23-5
