File: panel_rp2354_20x20_v0p2/panel_mcu.kicad_sch (KiCad schematic)
At the start: 32 parts, among them SW1 SW_Push, SW2 SW_Push, U1 APS6404L-3SQR, U2 RP2354B_80QFN, Y1 ABM8-272-T3

Commit message: Fixed ERC and DRC warnings
Parts:
- C1, C10, C11, C12, C13, C14, C15, C16, C17, C18, C2, C3, C6, C9: footprint Capacitor_SMD:C_0201_0603Metric -> panel_custom:C_0201_0603Metric
- C7, C8: footprint Capacitor_SMD:C_0402_1005Metric -> panel_custom:C_0402_1005Metric_4u7
- R1, R2, R3, R4, R5, R6, R7, R8: footprint Resistor_SMD:R_0201_0603Metric -> panel_custom:R_0201_0603Metric
- Y1: footprint Crystal:Crystal_SMD_3225-4Pin_3.2x2.5mm -> panel_custom:Crystal_SMD_3225-4Pin_3.2x2.5mm; symbol Device:Crystal_GND24 -> panel_custom:Crystal_GND24
Changed lines of the file:
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@@
 	(title_block
 		(title "G6 panel 45mm RP2354")
-		(date "2026-04-02")
+		(date "2026-04-03")
 		(rev "v0.2.0")
 		(company "IORodeo for Reiserlab @ Janelia")
@@
 			)
 		)
-		(property "Footprint" "Capacitor_SMD:C_0201_0603Metric"
+		(property "Footprint" "panel_custom:C_0201_0603Metric"
 			(at 44.45 117.8052 0)
 			(effects
@@
 			)
 		)
-		(property "Footprint" "Capacitor_SMD:C_0201_0603Metric"
+		(property "Footprint" "panel_custom:C_0201_0603Metric"
 			(at 44.45 127.9652 0)
 			(effects
@@
 			)
 		)
-		(property "Footprint" "Capacitor_SMD:C_0201_0603Metric"
+		(property "Footprint" "panel_custom:C_0201_0603Metric"
 			(at 258.7752 40.64 0)
 			(effects
@@
 			)
 		)
-		(property "Footprint" "Capacitor_SMD:C_0201_0603Metric"
+		(property "Footprint" "panel_custom:C_0201_0603Metric"
 			(at 270.2052 40.64 0)
 			(effects
@@
 			)
 		)
-		(property "Footprint" "Capacitor_SMD:C_0201_0603Metric"
+		(property "Footprint" "panel_custom:C_0201_0603Metric"
 			(at 281.6352 40.64 0)
 			(effects
@@
 			)
 		)
-		(property "Footprint" "Capacitor_SMD:C_0201_0603Metric"
+		(property "Footprint" "panel_custom:C_0201_0603Metric"
 			(at 293.0652 40.64 0)
 			(effects
@@
 			)
 		)
-		(property "Footprint" "Capacitor_SMD:C_0201_0603Metric"
+		(property "Footprint" "panel_custom:C_0201_0603Metric"
 			(at 304.4952 40.64 0)
 			(effects
@@
 			)
 		)
-		(property "Footprint" "Capacitor_SMD:C_0201_0603Metric"
+		(property "Footprint" "panel_custom:C_0201_0603Metric"
 			(at 315.9252 40.64 0)
 			(effects
@@
 	)
 	(symbol
-		(lib_id "Device:Crystal_GND24")
+		(lib_id "panel_custom:Crystal_GND24")
 		(at 63.5 121.92 270)
 		(unit 1)
@@
 			)
 		)
-		(property "Footprint" "Crystal:Crystal_SMD_3225-4Pin_3.2x2.5mm"
+		(property "Footprint" "panel_custom:Crystal_SMD_3225-4Pin_3.2x2.5mm"
 			(at 63.5 121.92 0)
 			(effects
@@
 		(pin "7"
 		)
+		(pin "9"
+		)
 		(instances
 			(project "panel_rp2354_20x20"
@@
 			)
 		)
-		(property "Footprint" "Capacitor_SMD:C_0201_0603Metric"
+		(property "Footprint" "panel_custom:C_0201_0603Metric"
 			(at 173.6852 40.64 0)
 			(effects
@@
 			)
 		)
-		(property "Footprint" "Resistor_SMD:R_0201_0603Metric"
+		(property "Footprint" "panel_custom:R_0201_0603Metric"
 			(at 256.54 64.262 90)
 			(effects
@@
 			)
 		)
-		(property "Footprint" "Capacitor_SMD:C_0201_0603Metric"
+		(property "Footprint" "panel_custom:C_0201_0603Metric"
 			(at 247.3452 40.64 0)
 			(effects
@@
 			)
 		)
-		(property "Footprint" "Capacitor_SMD:C_0201_0603Metric"
+		(property "Footprint" "panel_custom:C_0201_0603Metric"
 			(at 327.3552 40.64 0)
 			(effects
@@
 			)
 		)
-		(property "Footprint" "Resistor_SMD:R_0201_0603Metric"
+		(property "Footprint" "panel_custom:R_0201_0603Metric"
 			(at 70.358 160.02 90)
 			(effects
@@
 			)
 		)
-		(property "Footprint" "Capacitor_SMD:C_0402_1005Metric"
+		(property "Footprint" "panel_custom:C_0402_1005Metric_4u7"
 			(at 160.9852 69.85 0)
 			(effects
@@
 			)
 		)
-		(property "Footprint" "Resistor_SMD:R_0201_0603Metric"
+		(property "Footprint" "panel_custom:R_0201_0603Metric"
 			(at 60.96 168.402 90)
 			(effects
@@
 			)
 		)
-		(property "Footprint" "Resistor_SMD:R_0201_0603Metric"
+		(property "Footprint" "panel_custom:R_0201_0603Metric"
 			(at 81.28 125.222 90)
 			(effects
@@
 			)
 		)
-		(property "Footprint" "Capacitor_SMD:C_0201_0603Metric"
+		(property "Footprint" "panel_custom:C_0201_0603Metric"
 			(at 150.8252 40.64 0)
 			(effects
@@
 			)
 		)
-		(property "Footprint" "Capacitor_SMD:C_0201_0603Metric"
+		(property "Footprint" "panel_custom:C_0201_0603Metric"
 			(at 89.8652 80.01 0)
 			(effects
@@
 			)
 		)
-		(property "Footprint" "Capacitor_SMD:C_0402_1005Metric"
+		(property "Footprint" "panel_custom:C_0402_1005Metric_4u7"
 			(at 162.2552 40.64 0)
 			(effects
@@
 			)
 		)
-		(property "Footprint" "Capacitor_SMD:C_0201_0603Metric"
+		(property "Footprint" "panel_custom:C_0201_0603Metric"
 			(at 235.9152 40.64 0)
 			(effects
@@
 			)
 		)
-		(property "Footprint" "Resistor_SMD:R_0201_0603Metric"
+		(property "Footprint" "panel_custom:R_0201_0603Metric"
 			(at 50.8 205.232 90)
 			(effects
@@
 			)
 		)
-		(property "Footprint" "Resistor_SMD:R_0201_0603Metric"
+		(property "Footprint" "panel_custom:R_0201_0603Metric"
 			(at 148.59 62.738 90)
 			(effects
@@
 			)
 		)
-		(property "Footprint" "Resistor_SMD:R_0201_0603Metric"
+		(property "Footprint" "panel_custom:R_0201_0603Metric"
 			(at 256.54 73.152 90)
 			(effects
@@
 			)
 		)
-		(property "Footprint" "Resistor_SMD:R_0201_0603Metric"
+		(property "Footprint" "panel_custom:R_0201_0603Metric"
 			(at 50.038 57.15 90)
 			(effects
