File: panel_rp2354_20x20_v0p2/panel_usb_power.kicad_sch (KiCad schematic)
At the start: 4 parts, among them J1 Conn_01x04, U43 AP2112K-3.3

Commit message: Fixed ERC and DRC warnings
Parts:
- C67: footprint Capacitor_SMD:C_0402_1005Metric -> panel_custom:C_0402_1005Metric_NoSilk
- C68: footprint Capacitor_SMD:C_0402_1005Metric -> panel_custom:C_0402_1005Metric
- J1: symbol Connector_Generic:Conn_01x04 -> panel_custom:Conn_01x04_MP
- U43: footprint Package_TO_SOT_SMD:SOT-23-5 -> panel_custom:AP2112K-3.3_SOT-23-5; symbol Regulator_Linear:AP2112K-3.3 -> panel_custom:AP2112K-3.3
Changed lines of the file:
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@@
 	(title_block
 		(title "G6 panel 45mm RP2354")
-		(date "2026-04-02")
+		(date "2026-04-03")
 		(rev "v0.2.0")
 		(company "IORodeo for Reiserlab @ Janelia")
@@
 			)
 		)
-		(property "Footprint" "Capacitor_SMD:C_0402_1005Metric"
+		(property "Footprint" "panel_custom:C_0402_1005Metric_NoSilk"
 			(at 201.6252 57.15 0)
 			(effects
@@
 	)
 	(symbol
-		(lib_id "Connector_Generic:Conn_01x04")
+		(lib_id "panel_custom:Conn_01x04_MP")
 		(at 73.66 49.53 180)
 		(unit 1)
@@
 		(pin "4"
 		)
+		(pin "MP"
+		)
 		(instances
 			(project "panel_rp2354_20x20"
@@
 			)
 		)
-		(property "Footprint" "Capacitor_SMD:C_0402_1005Metric"
+		(property "Footprint" "panel_custom:C_0402_1005Metric"
 			(at 227.0252 57.15 0)
 			(effects
@@
 	)
 	(symbol
-		(lib_id "Regulator_Linear:AP2112K-3.3")
+		(lib_id "panel_custom:AP2112K-3.3")
 		(at 214.63 48.26 0)
 		(unit 1)
@@
 			)
 		)
-		(property "Footprint" "Package_TO_SOT_SMD:SOT-23-5"
+		(property "Footprint" "panel_custom:AP2112K-3.3_SOT-23-5"
 			(at 214.63 40.005 0)
 			(effects
